File: chunchunkb.kicad_pcb (KiCad board)
At the start: 2 copper layers, 152.4 x 142.8 mm, 124 parts, among them J1 BATT, J2 OLED, SW1 SW_Push, SW10 SW_Push, SW11 SW_Push, SW12 SW_Push, SW13 SW_Push, SW14 SW_Push, SW15 SW_Push, SW16 SW_Push, SW17 SW_Push, SW18 SW_Push, SW19 SW_Push, SW2 SW_Push, SW20 SW_Push, SW21 SW_Push, SW22 SW_Push, SW23 SW_Push, SW24 SW_Push, SW25 SW_Push, SW26 SW_Push, SW27 SW_Push, SW28 SW_Push, SW29 SW_Push, SW3 SW_Push, SW30 SW_Push, SW31 EC11, SW32 SW_Push, SW33 SW_Push, SW34 SW_Push, SW35 SW_Push, SW36 SW_Push, SW4 SW_Push, SW5 SW_Push, SW6 SW_Push, SW7 SW_Push, SW8 SW_Push, SW9 SW_Push

Commit message: wip
Parts:
- added LED36: YS-SK6812MINI-E, chunchunkb:YS-SK6812MINI-E, F.Cu at (76.2, 128.6)
- added RE1: EC11, chunchunkb:EC11_Switch, F.Cu at (552.5, -95.2)
- LED10, LED11, LED12, LED19, LED20, LED21, LED22, LED23, LED24, LED31, LED32, LED33, LED34, LED35, LED7, LED8, LED9: moved to F.Cu
- SW31: value EC11 -> SW_Push; footprint chunchunkb:EC11_Switch -> chunchunkb:MX-1U-Hotswap
- U1: footprint chunchunkb:ProMicro_DUAL -> chunchunkb:ProMicro_R
- moved H1 395.0 mm to (542.9, -143.9)
- moved H2 395.0 mm to (542.9, -138.8)
- moved H3 395.0 mm to (542.9, -133.7)
- moved H4 395.0 mm to (542.9, -128.6)
- moved JP6 376.7 mm to (522.5, -170.7)
- moved JP7 376.7 mm to (522.5, -167.8)
- moved JP8 376.7 mm to (522.5, -164.9)
- moved JP1 376.7 mm to (519.1, -170.7)
- moved JP2 376.7 mm to (519.1, -167.8)
- moved JP3 376.7 mm to (519.1, -164.9)
- moved JP4 376.7 mm to (519.1, -161.9)
- moved JP5 376.7 mm to (519.1, -159.0)
- moved SW_POWER1 350.8 mm to (519.1, -114.3)
- moved J1 334.0 mm to (504.8, -90.5)
- moved SW_RST1 313.4 mm to (485.8, -71.4)
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Connections:
- D1 pad 1: Net-(D1-K) -> ROW 0
- D1 pad 2: ROW 0 -> Net-(D1-A)
- D10 pad 1: Net-(D10-K) -> ROW 1
- D10 pad 2: ROW 1 -> Net-(D10-A)
- D11 pad 1: Net-(D11-K) -> ROW 1
- D11 pad 2: ROW 1 -> Net-(D11-A)
- D12 pad 1: Net-(D12-K) -> ROW 1
- D12 pad 2: ROW 1 -> Net-(D12-A)
- D13 pad 1: Net-(D13-K) -> ROW 2
- D13 pad 2: ROW 2 -> Net-(D13-A)
- D14 pad 1: Net-(D14-K) -> ROW 2
- D14 pad 2: ROW 2 -> Net-(D14-A)
- D15 pad 1: Net-(D15-K) -> ROW 2
- D15 pad 2: ROW 2 -> Net-(D15-A)
- D16 pad 1: Net-(D16-K) -> ROW 2
- D16 pad 2: ROW 2 -> Net-(D16-A)
- D17 pad 1: Net-(D17-K) -> ROW 2
- D17 pad 2: ROW 2 -> Net-(D17-A)
- D18 pad 1: Net-(D18-K) -> ROW 2
- D18 pad 2: ROW 2 -> Net-(D18-A)
- D19 pad 1: Net-(D19-K) -> ROW 3
- D19 pad 2: ROW 3 -> Net-(D19-A)
- D2 pad 1: Net-(D2-K) -> ROW 0
- D2 pad 2: ROW 0 -> Net-(D2-A)
- D20 pad 1: Net-(D20-K) -> ROW 3
- D20 pad 2: ROW 3 -> Net-(D20-A)
- D21 pad 1: Net-(D21-K) -> ROW 3
- D21 pad 2: ROW 3 -> Net-(D21-A)
- D22 pad 1: Net-(D22-K) -> ROW 3
- D22 pad 2: ROW 3 -> Net-(D22-A)
- D23 pad 1: Net-(D23-K) -> ROW 3
- D23 pad 2: ROW 3 -> Net-(D23-A)
- D24 pad 1: Net-(D24-K) -> ROW 3
- D24 pad 2: ROW 3 -> Net-(D24-A)
- D25 pad 1: Net-(D25-K) -> ROW 4
- D25 pad 2: ROW 4 -> Net-(D25-A)
- D26 pad 1: Net-(D26-K) -> ROW 4
- D26 pad 2: ROW 4 -> Net-(D26-A)
- D27 pad 1: Net-(D27-K) -> ROW 4
- D27 pad 2: ROW 4 -> Net-(D27-A)
- D28 pad 1: Net-(D28-K) -> ROW 4
- D28 pad 2: ROW 4 -> Net-(D28-A)
- D29 pad 1: Net-(D29-K) -> ROW 4
- D29 pad 2: ROW 4 -> Net-(D29-A)
- D3 pad 1: Net-(D3-K) -> ROW 0
- D3 pad 2: ROW 0 -> Net-(D3-A)
- D30 pad 1: Net-(D30-K) -> ROW 4
- D30 pad 2: ROW 4 -> Net-(D30-A)
- D31 pad 1: SW31A -> ROW 5
- D31 pad 2: ROW 5 -> SW31B
- D32 pad 1: Net-(D32-K) -> ROW 5
- D32 pad 2: ROW 5 -> Net-(D32-A)
- D33 pad 1: Net-(D33-K) -> ROW 5
- D33 pad 2: ROW 5 -> Net-(D33-A)
- D34 pad 1: Net-(D34-K) -> ROW 5
- D34 pad 2: ROW 5 -> Net-(D34-A)
- D35 pad 1: Net-(D35-K) -> ROW 5
- D35 pad 2: ROW 5 -> Net-(D35-A)
- D36 pad 1: Net-(D36-K) -> ROW 5
- D36 pad 2: ROW 5 -> Net-(D36-A)
- D4 pad 1: Net-(D4-K) -> ROW 0
- D4 pad 2: ROW 0 -> Net-(D4-A)
- D5 pad 1: Net-(D5-K) -> ROW 0
- D5 pad 2: ROW 0 -> Net-(D5-A)
- D6 pad 1: Net-(D6-K) -> ROW 0
- D6 pad 2: ROW 0 -> Net-(D6-A)
- D7 pad 1: Net-(D7-K) -> ROW 1
- D7 pad 2: ROW 1 -> Net-(D7-A)
- D8 pad 1: Net-(D8-K) -> ROW 1
- D8 pad 2: ROW 1 -> Net-(D8-A)
- D9 pad 1: Net-(D9-K) -> ROW 1
- D9 pad 2: ROW 1 -> Net-(D9-A)
- LED35 pad 2: unconnected-(LED35-DOUT-Pad2) -> Net-(LED35-DOUT)
- SW1 pad 1: Net-(D1-K) -> COL 0
- SW1 pad 2: COL 0 -> Net-(D1-A)
- SW10 pad 1: Net-(D10-K) -> COL 3
- SW10 pad 2: COL 3 -> Net-(D10-A)
- SW11 pad 1: Net-(D11-K) -> COL 4
- SW11 pad 2: COL 4 -> Net-(D11-A)
- SW12 pad 1: Net-(D12-K) -> COL 5
- SW12 pad 2: COL 5 -> Net-(D12-A)
- SW13 pad 1: Net-(D13-K) -> COL 0
- SW13 pad 2: COL 0 -> Net-(D13-A)
- SW14 pad 1: Net-(D14-K) -> COL 1
- SW14 pad 2: COL 1 -> Net-(D14-A)
- SW15 pad 1: Net-(D15-K) -> COL 2
- SW15 pad 2: COL 2 -> Net-(D15-A)
- SW16 pad 1: Net-(D16-K) -> COL 3
- SW16 pad 2: COL 3 -> Net-(D16-A)
- SW17 pad 1: Net-(D17-K) -> COL 4
- SW17 pad 2: COL 4 -> Net-(D17-A)
- SW18 pad 1: Net-(D18-K) -> COL 5
- SW18 pad 2: COL 5 -> Net-(D18-A)
- SW19 pad 1: Net-(D19-K) -> COL 0
- SW19 pad 2: COL 0 -> Net-(D19-A)
- SW2 pad 1: Net-(D2-K) -> COL 1
- SW2 pad 2: COL 1 -> Net-(D2-A)
- SW20 pad 1: Net-(D20-K) -> COL 1
- SW20 pad 2: COL 1 -> Net-(D20-A)
- SW21 pad 1: Net-(D21-K) -> COL 2
- SW21 pad 2: COL 2 -> Net-(D21-A)
- SW22 pad 1: Net-(D22-K) -> COL 3
- SW22 pad 2: COL 3 -> Net-(D22-A)
- SW23 pad 1: Net-(D23-K) -> COL 4
- SW23 pad 2: COL 4 -> Net-(D23-A)
- SW24 pad 1: Net-(D24-K) -> COL 5
- SW24 pad 2: COL 5 -> Net-(D24-A)
- SW25 pad 1: Net-(D25-K) -> COL 0
- SW25 pad 2: COL 0 -> Net-(D25-A)
- SW26 pad 1: Net-(D26-K) -> COL 1
- SW26 pad 2: COL 1 -> Net-(D26-A)
- SW27 pad 1: Net-(D27-K) -> COL 2
- SW27 pad 2: COL 2 -> Net-(D27-A)
- SW28 pad 1: Net-(D28-K) -> COL 3
- SW28 pad 2: COL 3 -> Net-(D28-A)
- SW29 pad 1: Net-(D29-K) -> COL 4
- SW29 pad 2: COL 4 -> Net-(D29-A)
- SW3 pad 1: Net-(D3-K) -> COL 2
- SW3 pad 2: COL 2 -> Net-(D3-A)
- SW30 pad 1: Net-(D30-K) -> COL 5
- SW30 pad 2: COL 5 -> Net-(D30-A)
- SW32 pad 1: Net-(D32-K) -> COL 1
- SW32 pad 2: COL 1 -> Net-(D32-A)
- SW33 pad 1: Net-(D33-K) -> COL 2
- SW33 pad 2: COL 2 -> Net-(D33-A)
- SW34 pad 1: Net-(D34-K) -> COL 3
- SW34 pad 2: COL 3 -> Net-(D34-A)
- SW35 pad 1: Net-(D35-K) -> COL 4
- SW35 pad 2: COL 4 -> Net-(D35-A)
- SW36 pad 1: Net-(D36-K) -> COL 5
- SW36 pad 2: COL 5 -> Net-(D36-A)
- SW4 pad 1: Net-(D4-K) -> COL 3
- SW4 pad 2: COL 3 -> Net-(D4-A)
- SW5 pad 1: Net-(D5-K) -> COL 4
- SW5 pad 2: COL 4 -> Net-(D5-A)
- SW6 pad 1: Net-(D6-K) -> COL 5
- SW6 pad 2: COL 5 -> Net-(D6-A)
- SW7 pad 1: Net-(D7-K) -> COL 0
- SW7 pad 2: COL 0 -> Net-(D7-A)
- SW8 pad 1: Net-(D8-K) -> COL 1
- SW8 pad 2: COL 1 -> Net-(D8-A)
- SW9 pad 1: Net-(D9-K) -> COL 2
- SW9 pad 2: COL 2 -> Net-(D9-A)
Routing:
- net VCC: track 265.0 -> 1077.2 mm, vias 6 -> 36
- net ROW 3: track 0.00 -> 175.7 mm, vias 0 -> 12
- net ROW 4: track 0.00 -> 169.2 mm, vias 0 -> 12
- net COL 3: track 0.00 -> 136.0 mm, vias 0 -> 5
- net COL 2: track 0.00 -> 136.0 mm, vias 0 -> 5
- net COL 1: track 0.00 -> 136.0 mm, vias 0 -> 5
- net COL 0: track 0.00 -> 136.0 mm, vias 0 -> 5
- net COL 5: track 0.00 -> 136.0 mm, vias 0 -> 5
- net COL 4: track 0.00 -> 136.0 mm, vias 0 -> 5
- net ROW 1: track 129.9 -> 175.7 mm, vias 6 -> 12
- net ROW 2: track 132.6 -> 169.2 mm, vias 6 -> 12
- net ROW 0: track 133.5 -> 169.4 mm, vias 6 -> 12
- net Net-(LED19-DOUT): track 0.00 -> 22.3 mm, vias 0 -> 2
- net Net-(LED20-DOUT): track 0.00 -> 22.3 mm, vias 0 -> 2
- net Net-(LED8-DOUT): track 0.00 -> 22.3 mm, vias 0 -> 2
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Other:
- board size 152.4 x 142.8 mm -> 157.2 x 138.1 mm

Commit message: wip
Parts:
- removed LED36: YS-SK6812MINI-E, chunchunkb:YS-SK6812MINI-E
- removed RE1: EC11, chunchunkb:EC11_Switch
- SW31: value SW_Push -> EC11; footprint chunchunkb:MX-1U-Hotswap -> chunchunkb:EC11_Switch
- U1: footprint chunchunkb:ProMicro_R -> chunchunkb:ProMicro_R2
- moved H4 526.9 mm to (85.7, 133.3)
- moved H1 499.4 mm to (85.7, 57.1)
- moved H3 449.8 mm to (181.0, 133.3)
- moved H2 411.6 mm to (181.0, 57.1)
- moved J1 348.8 mm to (164.0, -16.1)
- moved J2 348.8 mm to (81.0, -20.9)
- moved JP1 348.8 mm to (178.3, -96.3)
- moved JP2 348.8 mm to (178.3, -93.4)
- moved JP3 348.8 mm to (178.3, -90.5)
- moved JP4 348.8 mm to (178.3, -87.5)
- moved JP5 348.8 mm to (178.3, -84.6)
- moved JP6 348.8 mm to (181.7, -96.3)
- moved JP7 348.8 mm to (181.7, -93.4)
- moved JP8 348.8 mm to (181.7, -90.5)
- moved SW_POWER1 348.8 mm to (178.3, -39.9)
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- renumbered D31 to D1, D14 to D10, D8 to D11, D2 to D12, D33 to D13, D27 to D14, D21 to D15, D15 to D16, D9 to D17, D3 to D18, D34 to D19, D25 to D2, D28 to D20, D22 to D21, D16 to D22, D10 to D23, D4 to D24, D35 to D25, D29 to D26, D23 to D27, D17 to D28, D11 to D29, D19 to D3, D5 to D30, D36 to D31, D30 to D32, D24 to D33, D18 to D34, D12 to D35, D6 to D36, D13 to D4, D7 to D5, D1 to D6, D32 to D7, D26 to D8, D20 to D9
Connections:
- D1 pad 1: ROW 5 -> ROW 0
- D1 pad 2: SW31B -> Net-(D1-A)
- D10 pad 1: ROW 2 -> ROW 1
- D10 pad 2: Net-(D14-A) -> Net-(D10-A)
- D11 pad 2: Net-(D8-A) -> Net-(D11-A)
- D12 pad 1: ROW 0 -> ROW 1
- D12 pad 2: Net-(D2-A) -> Net-(D12-A)
- D13 pad 1: ROW 5 -> ROW 2
- D13 pad 2: Net-(D33-A) -> Net-(D13-A)
- D14 pad 1: ROW 4 -> ROW 2
- D14 pad 2: Net-(D27-A) -> Net-(D14-A)
- D15 pad 1: ROW 3 -> ROW 2
- D15 pad 2: Net-(D21-A) -> Net-(D15-A)
- D16 pad 2: Net-(D15-A) -> Net-(D16-A)
- D17 pad 1: ROW 1 -> ROW 2
- D17 pad 2: Net-(D9-A) -> Net-(D17-A)
- D18 pad 1: ROW 0 -> ROW 2
- D18 pad 2: Net-(D3-A) -> Net-(D18-A)
- D19 pad 1: ROW 5 -> ROW 3
- D19 pad 2: Net-(D34-A) -> Net-(D19-A)
- D2 pad 1: ROW 4 -> ROW 0
- D2 pad 2: Net-(D25-A) -> Net-(D2-A)
- D20 pad 1: ROW 4 -> ROW 3
- D20 pad 2: Net-(D28-A) -> Net-(D20-A)
- D21 pad 2: Net-(D22-A) -> Net-(D21-A)
- D22 pad 1: ROW 2 -> ROW 3
- D22 pad 2: Net-(D16-A) -> Net-(D22-A)
- D23 pad 1: ROW 1 -> ROW 3
- D23 pad 2: Net-(D10-A) -> Net-(D23-A)
- D24 pad 1: ROW 0 -> ROW 3
- D24 pad 2: Net-(D4-A) -> Net-(D24-A)
- D25 pad 1: ROW 5 -> ROW 4
- D25 pad 2: Net-(D35-A) -> Net-(D25-A)
- D26 pad 2: Net-(D29-A) -> Net-(D26-A)
- D27 pad 1: ROW 3 -> ROW 4
- D27 pad 2: Net-(D23-A) -> Net-(D27-A)
- D28 pad 1: ROW 2 -> ROW 4
- D28 pad 2: Net-(D17-A) -> Net-(D28-A)
- D29 pad 1: ROW 1 -> ROW 4
- D29 pad 2: Net-(D11-A) -> Net-(D29-A)
- D3 pad 1: ROW 3 -> ROW 0
- D3 pad 2: Net-(D19-A) -> Net-(D3-A)
- D30 pad 1: ROW 0 -> ROW 4
- D30 pad 2: Net-(D5-A) -> Net-(D30-A)
- D31 pad 2: Net-(D36-A) -> SW31B
- D32 pad 1: ROW 4 -> ROW 5
- D32 pad 2: Net-(D30-A) -> Net-(D32-A)
- D33 pad 1: ROW 3 -> ROW 5
- D33 pad 2: Net-(D24-A) -> Net-(D33-A)
- D34 pad 1: ROW 2 -> ROW 5
- D34 pad 2: Net-(D18-A) -> Net-(D34-A)
- D35 pad 1: ROW 1 -> ROW 5
- D35 pad 2: Net-(D12-A) -> Net-(D35-A)
- D36 pad 1: ROW 0 -> ROW 5
- D36 pad 2: Net-(D6-A) -> Net-(D36-A)
- D4 pad 1: ROW 2 -> ROW 0
- D4 pad 2: Net-(D13-A) -> Net-(D4-A)
- D5 pad 1: ROW 1 -> ROW 0
- D5 pad 2: Net-(D7-A) -> Net-(D5-A)
- D6 pad 2: Net-(D1-A) -> Net-(D6-A)
- D7 pad 1: ROW 5 -> ROW 1
- D7 pad 2: Net-(D32-A) -> Net-(D7-A)
- D8 pad 1: ROW 4 -> ROW 1
- D8 pad 2: Net-(D26-A) -> Net-(D8-A)
- D9 pad 1: ROW 3 -> ROW 1
- D9 pad 2: Net-(D20-A) -> Net-(D9-A)
- LED35 pad 2: Net-(LED35-DOUT) -> unconnected-(LED35-DOUT-Pad2)
Routing:
- net ROW 5: track 12.0 -> 96.7 mm, vias 0 -> 5
- net ROW 1: track 175.7 -> 113.6 mm, vias 12 -> 6
- net ROW 3: track 175.7 -> 114.2 mm, vias 12 -> 6
- net COL 1: track 136.0 -> 192.6 mm, vias 5 -> 8
- net ROW 0: track 169.4 -> 114.2 mm, vias 12 -> 6
- net ROW 2: track 169.2 -> 114.5 mm, vias 12 -> 6
- net ROW 4: track 169.2 -> 115.7 mm, vias 12 -> 6
- net COL 2: track 136.0 -> 186.3 mm, vias 5 -> 8
- net COL 3: track 136.0 -> 186.3 mm, vias 5 -> 8
- net COL 4: track 136.0 -> 185.8 mm, vias 5 -> 8
- net COL 5: track 136.0 -> 183.2 mm, vias 5 -> 8
- net VCC: track 1077.2 -> 1034.1 mm, vias 36 -> 35
- net Net-(LED18-DOUT): track 0.00 -> 35.2 mm, vias 0 -> 4
- net Net-(LED6-DOUT): track 0.00 -> 35.2 mm, vias 0 -> 4
- net LED: track 19.9 -> 0.00 mm, vias 1 -> 0
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