File: chunchunkb.kicad_pcb (KiCad board)
At the start: 2 copper layers, 157.2 x 138.1 mm, 124 parts, among them J1 BATT, J2 OLED, SW1 SW_Push, SW10 SW_Push, SW11 SW_Push, SW12 SW_Push, SW13 SW_Push, SW14 SW_Push, SW15 SW_Push, SW16 SW_Push, SW17 SW_Push, SW18 SW_Push, SW19 SW_Push, SW2 SW_Push, SW20 SW_Push, SW21 SW_Push, SW22 SW_Push, SW23 SW_Push, SW24 SW_Push, SW25 SW_Push, SW26 SW_Push, SW27 SW_Push, SW28 SW_Push, SW29 SW_Push, SW3 SW_Push, SW30 SW_Push, SW31 EC11, SW32 SW_Push, SW33 SW_Push, SW34 SW_Push, SW35 SW_Push, SW36 SW_Push, SW4 SW_Push, SW5 SW_Push, SW6 SW_Push, SW7 SW_Push, SW8 SW_Push, SW9 SW_Push

Commit message: snapshot
Parts:
- JP5, JP6, JP7, JP8: moved to B.Cu
- moved JP6 201.0 mm to (71.4, 71.8), turned to 90 degrees
- moved JP7 196.6 mm to (75.0, 71.8), turned to 90 degrees
- moved JP1 196.2 mm to (77.1, 71.8), turned to 90 degrees
- moved JP2 194.8 mm to (75.0, 71.8), turned to 90 degrees
- moved JP3 194.3 mm to (71.4, 71.8), turned to 90 degrees
- moved JP8 193.1 mm to (77.1, 71.8), turned to 90 degrees
- moved JP4 193.0 mm to (69.4, 71.8), turned to 90 degrees
- moved JP5 190.6 mm to (69.4, 71.8), turned to 90 degrees
- moved SW_POWER1 130.8 mm to (73.3, 38.1), turned to 180 degrees
- moved J2 79.6 mm to (73.2, 58.3)
- moved U1 6.20 mm to (73.2, 55.1)
Connections:
- JP3 pad 2: MOSI/SDA -> SCK/SCL
- JP4 pad 2: SCK/SCL -> MOSI/SDA
- JP7 pad 2: MOSI/SDA -> SCK/SCL
- JP8 pad 2: SCK/SCL -> MOSI/SDA
Routing:
- net Net-(LED30-DOUT): track 0.00 -> 62.3 mm, vias 0 -> 3
- net CS: track 0.00 -> 52.6 mm, vias 0 -> 2
- net MOSI/SDA: track 0.00 -> 43.4 mm, vias 0 -> 2
- net VCC: track 1034.1 -> 1070.0 mm, vias 35 -> 36
- net SCK/SCL: track 0.00 -> 34.1 mm, vias 0 -> 2
- net ROW 5: track 96.7 -> 115.1 mm
- net COL 5: track 183.2 -> 200.3 mm
- net Net-(LED12-DOUT): track 0.00 -> 15.8 mm, vias 0 -> 2
- net ROW 4: track 115.7 -> 131.0 mm
- net COL 4: track 185.8 -> 200.6 mm
- net COL 3: track 186.3 -> 199.5 mm
- net ROW 3: track 114.2 -> 127.0 mm
- net COL 2: track 186.3 -> 198.3 mm
- net COL 1: track 192.6 -> 204.7 mm
- net RESET: track 0.00 -> 12.0 mm
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
Commit message: snapshot
Parts:
- D1, D10, D11, D12, D13, D14, D15, D16, D17, D18, D19, D2, D20, D21, D22, D23, D24, D25, D26, D27, D28, D29, D3, D30, D31, D32, D33, D34, D35, D36, D4, D5, D6, D7, D8, D9: footprint chunchunkb:D_SOD-123 -> chunchunkb:crkbd-diode
- U1: footprint chunchunkb:ProMicro_R2 -> chunchunkb:ProMicro DUAL
- moved J1 107.9 mm to (92.5, 64.7)
- moved SW_RST1 84.9 mm to (84.2, 62.2), turned to -90 degrees
- moved LED32 30.5 mm to (152.4, 123.8)
- moved LED33 30.5 mm to (133.3, 123.8)
- moved LED34 30.5 mm to (114.3, 123.8)
- moved LED35 30.5 mm to (95.2, 123.8)
- moved LED31 30.5 mm to (171.4, 123.8)
- moved LED23 30.5 mm to (133.3, 85.7)
- moved LED11 30.5 mm to (133.3, 47.6)
- moved LED2 30.5 mm to (133.3, 28.6)
- moved LED19 30.5 mm to (209.5, 85.7)
- moved LED20 30.5 mm to (190.5, 85.7)
- moved LED21 30.5 mm to (171.4, 85.7)
- moved LED22 30.5 mm to (152.4, 85.7)
- moved LED24 30.5 mm to (114.3, 85.7)
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Routing:
- net COL 5: track 200.3 -> 346.9 mm, vias 8 -> 10
- net COL 4: track 200.6 -> 319.0 mm, vias 8 -> 10
- net ROW 5: track 115.1 -> 217.3 mm, vias 5 -> 8
- net VCC: track 1070.0 -> 1168.6 mm, vias 36 -> 39
- net COL 3: track 199.5 -> 293.0 mm, vias 8 -> 10
- net ENC A: track 12.0 -> 96.6 mm, vias 0 -> 1
- net ENC B: track 12.0 -> 88.6 mm, vias 0 -> 1
- net ROW 4: track 131.0 -> 205.7 mm, vias 6 -> 8
- net COL 2: track 198.3 -> 268.5 mm, vias 8 -> 10
- net COL 0: track 135.5 -> 205.3 mm, vias 5 -> 9
- net ROW 3: track 127.0 -> 187.1 mm, vias 6 -> 8
- net Net-(J1-Pin_1): track 0.00 -> 58.3 mm, vias 0 -> 2
- net ROW 2: track 126.6 -> 168.7 mm, vias 6 -> 8
- net COL 1: track 204.7 -> 244.7 mm, vias 8 -> 10
- net GND: track 0.00 -> 38.5 mm, vias 0 -> 1
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Other:
- board size 157.2 x 138.1 mm -> 143.7 x 121.4 mm
- rule pad_to_mask_clearance: 0.2 -> 0

Commit message: snapshot
Routing:
- net COL 1: track 244.7 -> 243.8 mm
- net COL 0: track 205.3 -> 205.9 mm
- net COL 3: track 293.0 -> 293.6 mm
Changed lines of the file:
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@@
 	)
 	(segment
-		(start 176.770944 22.882792)
-		(end 178.295944 24.407792)
-		(width 0.25)
-		(layer "F.Cu")
-		(net "COL 3")
-	)
-	(segment
 		(start 168.473296 119.0624)
 		(end 161.933948 119.0624)
@@
 	)
 	(segment
-		(start 97.667888 22.882792)
-		(end 176.770944 22.882792)
-		(width 0.25)
-		(layer "F.Cu")
-		(net "COL 3")
-	)
-	(segment
 		(start 177.127806 54.580424)
 		(end 178.427806 53.280424)
@@
 	)
 	(segment
-		(start 96.142888 24.407792)
-		(end 97.667888 22.882792)
+		(start 177.663912 22.882792)
+		(end 178.444772 23.663652)
 		(width 0.25)
 		(layer "F.Cu")
@@
 	)
 	(segment
+		(start 97.667888 22.882792)
+		(end 177.663912 22.882792)
+		(width 0.25)
+		(layer "F.Cu")
+		(net "COL 3")
+	)
+	(segment
+		(start 96.142888 24.407792)
+		(end 97.667888 22.882792)
+		(width 0.25)
+		(layer "F.Cu")
+		(net "COL 3")
+	)
+	(segment
 		(start 177.127806 73.630408)
 		(end 178.427806 72.330408)
@@
 	)
 	(via
-		(at 178.295944 24.407792)
+		(at 178.444772 23.663652)
 		(size 0.6)
 		(drill 0.3)
@@
 	)
 	(segment
+		(start 178.427806 23.680618)
+		(end 178.427806 34.23044)
+		(width 0.25)
+		(layer "B.Cu")
+		(net "COL 3")
+	)
+	(segment
 		(start 178.427806 35.81942)
 		(end 178.427806 53.280424)
@@
 	)
 	(segment
-		(start 178.427806 24.539654)
-		(end 178.427806 34.23044)
-		(width 0.25)
-		(layer "B.Cu")
-		(net "COL 3")
-	)
-	(segment
-		(start 178.295944 24.407792)
-		(end 178.427806 24.539654)
-		(width 0.25)
-		(layer "B.Cu")
-		(net "COL 3")
-	)
-	(segment
 		(start 178.427806 112.01942)
 		(end 178.427806 114.146282)
@@
 	)
 	(segment
+		(start 178.444772 23.663652)
+		(end 178.427806 23.680618)
+		(width 0.25)
+		(layer "B.Cu")
+		(net "COL 3")
+	)
+	(segment
 		(start 142.87488 119.955368)
 		(end 140.35 122.480248)
@@
 	)
 	(segment
-		(start 140.327806 25.43259)
-		(end 138.678008 23.782792)
-		(width 0.25)
-		(layer "F.Cu")
-		(net "COL 1")
-	)
-	(segment
 		(start 139.027806 73.630408)
 		(end 140.327806 72.330408)
@@
 	)
 	(segment
-		(start 98.553824 23.782792)
-		(end 97.928824 24.407792)
+		(start 139.027806 111.730376)
+		(end 140.327806 110.430376)
 		(width 0.25)
 		(layer "F.Cu")
@@
 	)
 	(segment
-		(start 139.027806 111.730376)
-		(end 140.327806 110.430376)
+		(start 122.941012 119.955368)
+		(end 107.751472 119.955368)
 		(width 0.25)
 		(layer "F.Cu")
@@
 	)
 	(segment
-		(start 138.678008 23.782792)
+		(start 139.702806 23.782792)
 		(end 98.553824 23.782792)
 		(width 0.25)
@@
 	)
 	(segment
-		(start 122.941012 119.955368)
-		(end 107.751472 119.955368)
+		(start 98.553824 23.782792)
+		(end 97.928824 24.407792)
 		(width 0.25)
 		(layer "F.Cu")
@@
 	)
 	(segment
+		(start 140.327806 24.407792)
+		(end 139.702806 23.782792)
+		(width 0.25)
+		(layer "F.Cu")
+		(net "COL 1")
+	)
+	(segment
 		(start 139.027806 35.53044)
 		(end 140.327806 34.23044)
@@
 	)
 	(via
-		(at 140.327806 25.43259)
+		(at 140.327806 24.407792)
 		(size 0.6)
 		(drill 0.3)
@@
 	)
 	(segment
+		(start 140.327806 114.168074)
+		(end 135.43348 119.0624)
+		(width 0.25)
+		(layer "B.Cu")
+		(net "COL 1")
+	)
+	(segment
 		(start 140.327806 72.330408)
 		(end 140.327806 91.380392)
@@
 	)
 	(segment
+		(start 140.327806 24.407792)
+		(end 140.327806 34.23044)
+		(width 0.25)
+		(layer "B.Cu")
+		(net "COL 1")
+	)
+	(segment
 		(start 140.327806 53.280424)
 		(end 140.327806 72.330408)
@@
 	)
 	(segment
-		(start 138.112384 119.0624)
+		(start 135.43348 119.0624)
 		(end 130.373328 119.0624)
 		(width 0.25)
@@
 	)
 	(segment
-		(start 140.327806 25.43259)
-		(end 140.327806 34.23044)
-		(width 0.25)
-		(layer "B.Cu")
-		(net "COL 1")
-	)
-	(segment
 		(start 140.327806 35.81942)
 		(end 140.327806 53.280424)
@@
 	)
 	(segment
-		(start 140.327806 116.846978)
-		(end 138.112384 119.0624)
-		(width 0.25)
-		(layer "B.Cu")
-		(net "COL 1")
-	)
-	(segment
 		(start 140.327806 112.01942)
-		(end 140.327806 116.846978)
+		(end 140.327806 114.168074)
 		(width 0.25)
 		(layer "B.Cu")
@@
 	)
 	(segment
-		(start 98.821792 24.407792)
-		(end 119.944214 24.407792)
+		(start 120.98015 24.407792)
+		(end 98.821792 24.407792)
 		(width 0.25)
 		(layer "F.Cu")
@@
 	)
 	(segment
-		(start 119.944214 24.407792)
-		(end 121.277806 25.741384)
-		(width 0.25)
-		(layer "F.Cu")
-		(net "COL 0")
-	)
-	(segment
 		(start 119.977806 73.630408)
 		(end 121.277806 72.330408)
@@
 	)
 	(segment
+		(start 121.277806 24.705448)
+		(end 120.98015 24.407792)
+		(width 0.25)
+		(layer "F.Cu")
+		(net "COL 0")
+	)
+	(segment
 		(start 119.977806 54.580424)
 		(end 121.277806 53.280424)
@@
 	)
 	(via
-		(at 121.277806 25.741384)
+		(at 121.277806 24.705448)
 		(size 0.6)
 		(drill 0.3)
@@
 	)
 	(segment
-		(start 121.277806 25.741384)
-		(end 121.277806 34.23044)
-		(width 0.25)
-		(layer "B.Cu")
-		(net "COL 0")
-	)
-	(segment
 		(start 84.975704 103.751221)
 		(end 89.607477 99.119448)
@@
 		(width 0.25)
 		(layer "B.Cu")
+		(net "COL 0")
+	)
+	(segment
+		(start 121.277806 24.705448)
+		(end 121.277806 34.23044)
+		(width 0.25)
+		(layer "B.Cu")
